File: pcb/excelsior.kicad_pcb (KiCad board)
At the start: 2 copper layers, 12 parts, among them J1 USB_Hub4_FDD, J2 USB_Hub3, J3 USB_Hub2, J4 Conn_01x40_Socket, P1 Host_Port, P2 Left_Peripheral, P3 Right_Peripheral, U1 kb2040, U2 MCP23017_SO, U3 CH334R

Commit message: Continue work on PCB design.
Parts:
- removed REF** (x2): MountingHole_2.2mm_M2_DIN965_Pad_TopBottom, MountingHole:MountingHole_2.2mm_M2_DIN965_Pad_TopBottom
- added SW1: SW_Push, Button_Switch_SMD:SW_SPST_EVPBF, F.Cu at (117.0, 25.5)
- J1, J2, J3: footprint Connector_USB:USB_A_TE_292303-7_Horizontal -> Connector_USB:USB_A_Molex_67643_Horizontal
- P1, P2, P3: footprint Connector_USB:USB_C_Receptacle_Molex_105450-0101 -> Connector_USB:USB_C_Receptacle_GCT_USB4085
- U2: footprint Package_SO:SOIC-28W_7.5x17.9mm_P1.27mm -> Package_DIP:DIP-28_W7.62mm
- moved J4 122.0 mm to (22.0, 48.0), turned to 90 degrees
- moved P3 50.0 mm to (314.0, 38.0)
- moved P1 45.7 mm to (310.0, 26.0)
- moved P2 38.9 mm to (26.0, 32.0)
- moved J1 33.7 mm to (280.0, 30.0)
- moved J2 31.6 mm to (260.0, 30.0)
- moved J3 29.6 mm to (240.0, 30.0)
- moved U1 28.6 mm to (200.6, 33.4), turned to -90 degrees
- moved U3 15.8 mm to (259.9, 44.5)
- moved U2 10.1 mm to (71.5, 41.6), turned to 90 degrees
Connections:
- net Net-(J1-D+) renamed DM4+
- net Net-(J1-D-) renamed DM4-
- net Net-(J2-D+) renamed DM3+
- net Net-(J2-D-) renamed DM3-
- net Net-(J3-D+) renamed DM2+
- net Net-(J3-D-) renamed DM2-
- net Net-(U1-D+) renamed DM1+
- net Net-(U1-D-) renamed DM1-
- J1 pad 1: Net-(J1-VBUS) -> VBUS
- J1 pad 4: Net-(J1-GND) -> GND
- J1 pad 5: Net-(J1-GND) -> GND
- J2 pad 1: Net-(J1-VBUS) -> VBUS
- J2 pad 4: Net-(J1-GND) -> GND
- J2 pad 5: Net-(J1-GND) -> GND
- J3 pad 1: Net-(J1-VBUS) -> VBUS
- J3 pad 4: Net-(J1-GND) -> GND
- J3 pad 5: Net-(J1-GND) -> GND
- J4 pad 1: unconnected-(J4-Pin_1-Pad1) -> VBUS
- J4 pad 10: Net-(J4-Pin_10) -> GND
- J4 pad 11: Net-(J4-Pin_11) -> IO_07
- J4 pad 12: Net-(J4-Pin_12) -> IO_08
- J4 pad 13: Net-(J4-Pin_13) -> IO_09
- J4 pad 14: Net-(J4-Pin_14) -> IO_10
- J4 pad 15: Net-(J4-Pin_15) -> IO_11
- J4 pad 16: Net-(J4-Pin_16) -> IO_12
- J4 pad 17: Net-(J4-Pin_17) -> IO_13
- J4 pad 18: Net-(J4-Pin_18) -> GND
- J4 pad 19: Net-(J4-Pin_19) -> IO_14
- J4 pad 2: unconnected-(J4-Pin_2-Pad2) -> GND
- J4 pad 20: Net-(J4-Pin_20) -> IO_15
- J4 pad 21: Net-(J4-Pin_21) -> IO_16
- J4 pad 22: Net-(J4-Pin_22) -> IO_17
- J4 pad 23: Net-(J4-Pin_23) -> IO_18
- J4 pad 24: Net-(J4-Pin_24) -> IO_19
- J4 pad 25: Net-(J4-Pin_25) -> IO_20
- J4 pad 26: Net-(J4-Pin_26) -> IO_21
- J4 pad 27: Net-(J4-Pin_27) -> IO_22
- J4 pad 28: Net-(J4-Pin_28) -> IO_23
- J4 pad 29: Net-(J4-Pin_29) -> IO_24
- J4 pad 3: unconnected-(J4-Pin_3-Pad3) -> IO_00
- J4 pad 30: Net-(J4-Pin_30) -> IO_25
- J4 pad 31: Net-(J4-Pin_31) -> GND
- J4 pad 32: Net-(J4-Pin_32) -> IO_26
- J4 pad 33: Net-(J4-Pin_33) -> IO_27
- J4 pad 34: Net-(J4-Pin_34) -> IO_28
- J4 pad 35: Net-(J4-Pin_35) -> SCK
- J4 pad 36: Net-(J1-GND) -> SDA
- J4 pad 37: unconnected-(J4-Pin_37-Pad37) -> MISO
- J4 pad 38: unconnected-(J4-Pin_38-Pad38) -> MOSI
- J4 pad 39: unconnected-(J4-Pin_39-Pad39) -> GND
- J4 pad 4: Net-(J1-VBUS) -> IO_01
- J4 pad 40: unconnected-(J4-Pin_40-Pad40) -> VBUS
- J4 pad 5: Net-(J4-Pin_5) -> IO_02
- J4 pad 6: Net-(J4-Pin_6) -> IO_03
- J4 pad 7: Net-(J4-Pin_7) -> IO_04
- J4 pad 8: Net-(J4-Pin_8) -> IO_05
- J4 pad 9: Net-(J4-Pin_9) -> IO_06
- P1 pad A1: Net-(J1-GND) -> GND
- P1 pad A12: Net-(J1-GND) -> GND
- P1 pad A4: Net-(J1-VBUS) -> VBUS
- P1 pad A6: Net-(U3-DPU+) -> HOST_D+
- P1 pad A7: Net-(U3-DMU-) -> HOST_D-
- P1 pad A8: unconnected-(P1-SBU1-PadA8) -> (no net)
- P1 pad A9: Net-(J1-VBUS) -> VBUS
- P1 pad B1: Net-(J1-GND) -> GND
- P1 pad B12: Net-(J1-GND) -> GND
- P1 pad B4: Net-(J1-VBUS) -> VBUS
- P1 pad B6: Net-(U3-DPU+) -> (no net)
- P1 pad B7: Net-(U3-DMU-) -> (no net)
- P1 pad B8: unconnected-(P1-SBU2-PadB8) -> (no net)
- P1 pad B9: Net-(J1-VBUS) -> VBUS
- P1 pad S1: Net-(J1-GND) -> GND
- P2 pad A1: Net-(J1-GND) -> GND
- P2 pad A12: Net-(J1-GND) -> GND
- P2 pad A4: Net-(J1-VBUS) -> VBUS
- P2 pad A6: Net-(U1-A0/26) -> SCK
- P2 pad A7: Net-(U1-SCK/18) -> SDA
- P2 pad A8: unconnected-(P2-SBU1-PadA8) -> (no net)
- P2 pad A9: Net-(J1-VBUS) -> VBUS
- P2 pad B1: Net-(J1-GND) -> GND
- P2 pad B12: Net-(J1-GND) -> GND
- P2 pad B4: Net-(J1-VBUS) -> VBUS
- P2 pad B6: Net-(U1-A0/26) -> (no net)
- P2 pad B7: Net-(U1-SCK/18) -> (no net)
- P2 pad B8: unconnected-(P2-SBU2-PadB8) -> (no net)
- P2 pad B9: Net-(J1-VBUS) -> VBUS
- P2 pad S1: Net-(J1-GND) -> GND
- P3 pad A1: Net-(J1-GND) -> GND
- P3 pad A12: Net-(J1-GND) -> GND
- P3 pad A4: Net-(J1-VBUS) -> VBUS
- P3 pad A6: Net-(U1-A0/26) -> SCK
- P3 pad A7: Net-(U1-SCK/18) -> SDA
- P3 pad A8: unconnected-(P3-SBU1-PadA8) -> (no net)
- P3 pad A9: Net-(J1-VBUS) -> VBUS
- P3 pad B1: Net-(J1-GND) -> GND
- P3 pad B12: Net-(J1-GND) -> GND
- P3 pad B4: Net-(J1-VBUS) -> VBUS
- P3 pad B6: Net-(U1-A0/26) -> (no net)
- P3 pad B7: Net-(U1-SCK/18) -> (no net)
- P3 pad B8: unconnected-(P3-SBU2-PadB8) -> (no net)
- P3 pad B9: Net-(J1-VBUS) -> VBUS
- P3 pad S1: Net-(J1-GND) -> GND
- U1 pad 10: Net-(J4-Pin_11) -> IO_06
- U1 pad 11: Net-(J4-Pin_12) -> IO_07
- U1 pad 12: Net-(J4-Pin_13) -> IO_08
- U1 pad 13: Net-(J4-Pin_14) -> IO_09
- U1 pad 15: Net-(J1-VBUS) -> VBUS
- U1 pad 16: Net-(J1-GND) -> GND
- U1 pad 19: Net-(J4-Pin_19) -> IO_10
- U1 pad 2: Net-(J4-Pin_5) -> IO_00
- U1 pad 20: Net-(J4-Pin_18) -> IO_11
- U1 pad 22: Net-(U1-A0/26) -> SDA
- U1 pad 23: Net-(U1-SCK/18) -> SCK
- U1 pad 24: Net-(J4-Pin_17) -> MISO
- U1 pad 25: Net-(J4-Pin_16) -> MOSI
- U1 pad 26: Net-(J4-Pin_15) -> IO_12
- U1 pad 3: Net-(J4-Pin_6) -> IO_01
- U1 pad 4: Net-(J1-GND) -> GND
- U1 pad 5: Net-(J1-GND) -> GND
- U1 pad 6: Net-(J4-Pin_7) -> IO_02
- U1 pad 7: Net-(J4-Pin_8) -> IO_03
- U1 pad 8: Net-(J4-Pin_9) -> IO_04
- U1 pad 9: Net-(J4-Pin_10) -> IO_05
- U2 pad 1: Net-(J4-Pin_35) -> IO_13
- U2 pad 10: Net-(J1-GND) -> GND
- U2 pad 12: Net-(U1-SCK/18) -> SCK
- U2 pad 13: Net-(U1-A0/26) -> SDA
- U2 pad 15: Net-(J1-GND) -> GND
- U2 pad 16: Net-(J1-GND) -> GND
- U2 pad 17: Net-(J1-GND) -> GND
- U2 pad 18: Net-(J1-GND) -> RESET
- U2 pad 2: Net-(J4-Pin_34) -> IO_14
- U2 pad 21: Net-(J4-Pin_27) -> IO_21
- U2 pad 22: Net-(J4-Pin_26) -> IO_22
- U2 pad 23: Net-(J4-Pin_25) -> IO_23
- U2 pad 24: Net-(J4-Pin_24) -> IO_24
- U2 pad 25: Net-(J4-Pin_23) -> IO_25
- U2 pad 26: Net-(J4-Pin_22) -> IO_26
- U2 pad 27: Net-(J4-Pin_21) -> IO_27
- U2 pad 28: Net-(J4-Pin_20) -> IO_28
- U2 pad 3: Net-(J4-Pin_33) -> IO_15
- U2 pad 4: Net-(J4-Pin_32) -> IO_16
- U2 pad 5: Net-(J4-Pin_31) -> IO_17
- U2 pad 6: Net-(J4-Pin_30) -> IO_18
- U2 pad 7: Net-(J4-Pin_29) -> IO_19
- U2 pad 8: Net-(J4-Pin_28) -> IO_20
- U2 pad 9: Net-(J1-VBUS) -> VBUS
- U3 pad 10: Net-(U3-DMU-) -> HOST_D-
- U3 pad 11: Net-(U3-DPU+) -> HOST_D+
- U3 pad 12: Net-(J1-VBUS) -> VBUS
- U3 pad 14: Net-(J1-GND) -> GND
- U3 pad 9: unconnected-(U3-~{RESET}/CDP-Pad9) -> RESET
Routing:
- net Net-(J1-VBUS): track 565.2 -> 0.00 mm, vias 3 -> 0
- net VBUS: track 0.00 -> 400.0 mm, vias 0 -> 1
- net Net-(U1-SCK/18): track 352.5 -> 0.00 mm, vias 2 -> 0
- net Net-(U1-A0/26): track 348.8 -> 0.00 mm, vias 2 -> 0
- net RESET: track 0.00 -> 171.7 mm
- net SCK: track 0.00 -> 137.5 mm
- net SDA: track 0.00 -> 135.0 mm
- net Net-(J4-Pin_15): track 95.2 -> 0.00 mm
- net Net-(J4-Pin_17): track 95.2 -> 0.00 mm
- net Net-(J4-Pin_16): track 95.2 -> 0.00 mm
- net Net-(J4-Pin_14): track 90.3 -> 0.00 mm
- net Net-(J4-Pin_19): track 87.6 -> 0.00 mm
- net Net-(J4-Pin_18): track 87.6 -> 0.00 mm
- net Net-(J4-Pin_13): track 84.9 -> 0.00 mm
- net Net-(J4-Pin_12): track 79.5 -> 0.00 mm
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- added copper zone on B.Cu, net GND
- added copper zone on F.Cu, net GND
- removed copper zone on B.Cu, net Net-(J1-GND)
- removed copper zone on F.Cu, net Net-(J1-GND)
Other:
- board outline added: 300 x 30 mm

Commit message: Continue work on PCBs, add Gerber files.
Parts:
- added REF**: MountingHole_2.2mm_M2_DIN965_Pad, MountingHole:MountingHole_2.2mm_M2_DIN965_Pad, F.Cu at (316.0, 24.0)
- added REF**: MountingHole_2.2mm_M2_DIN965_Pad, MountingHole:MountingHole_2.2mm_M2_DIN965_Pad, F.Cu at (316.0, 46.0)
- added REF**: MountingHole_2.2mm_M2_DIN965_Pad, MountingHole:MountingHole_2.2mm_M2_DIN965_Pad, F.Cu at (24.0, 46.0)
- added REF**: MountingHole_2.2mm_M2_DIN965_Pad, MountingHole:MountingHole_2.2mm_M2_DIN965_Pad, F.Cu at (24.0, 24.0)
- U2: footprint Package_DIP:DIP-28_W7.62mm -> Package_SO:SOIC-28W_7.5x17.9mm_P1.27mm
- moved U2 118.6 mm to (189.8, 33.9)
- moved J4 98.5 mm to (120.5, 48.0)
- moved SW1 96.2 mm to (213.0, 31.5)
- moved U1 61.9 mm to (138.7, 33.0), turned to 90 degrees
- moved U3 8.39 mm to (256.0, 37.0)
Connections:
- J4 pad 35: SCK -> MOSI
- J4 pad 37: MISO -> SCK
- J4 pad 38: MOSI -> MISO
- P1 pad A8: (no net) -> unconnected-(P1-SBU1-PadA8)
- P1 pad B6: (no net) -> HOST_D+
- P1 pad B7: (no net) -> HOST_D-
- P1 pad B8: (no net) -> unconnected-(P1-SBU2-PadB8)
- P2 pad A5: unconnected-(P2-CC-PadA5) -> MISO
- P2 pad A8: (no net) -> MOSI
- P2 pad B5: unconnected-(P2-VCONN-PadB5) -> MISO
- P2 pad B6: (no net) -> SCK
- P2 pad B7: (no net) -> SDA
- P2 pad B8: (no net) -> MOSI
- P3 pad A5: unconnected-(P3-CC-PadA5) -> MISO
- P3 pad A8: (no net) -> MOSI
- P3 pad B5: unconnected-(P3-VCONN-PadB5) -> MISO
- P3 pad B6: (no net) -> SCK
- P3 pad B7: (no net) -> SDA
- P3 pad B8: (no net) -> MOSI
Routing:
- net MOSI: track 0.00 -> 346.6 mm, vias 0 -> 3
- net MISO: track 0.00 -> 343.9 mm
- net SDA: track 135.0 -> 321.5 mm, vias 0 -> 1
- net SCK: track 137.5 -> 315.3 mm, vias 0 -> 1
- net RESET: track 171.7 -> 69.1 mm, vias 0 -> 2
- net DM1-: track 44.8 -> 145.1 mm
- net DM1+: track 62.2 -> 145.1 mm
- net Net-(U1-A1/27): track 107.8 -> 51.1 mm, vias 0 -> 1
- net IO_12: track 0.00 -> 38.5 mm, vias 0 -> 1
- net IO_21: track 55.0 -> 22.0 mm
- net IO_11: track 0.00 -> 29.3 mm
- net IO_10: track 0.00 -> 29.3 mm
- net IO_22: track 53.7 -> 26.7 mm
- net IO_23: track 52.3 -> 29.1 mm
- net IO_24: track 51.0 -> 31.4 mm
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
Commit message: Continue work on PCBs.
Parts:
- removed J1: USB_Hub4_FDD, Connector_USB:USB_A_Molex_67643_Horizontal
- removed J2: USB_Hub3, Connector_USB:USB_A_Molex_67643_Horizontal
- removed J3: USB_Hub2, Connector_USB:USB_A_Molex_67643_Horizontal
- removed J4: Conn_01x40_Socket, Connector_PinHeader_2.54mm:PinHeader_1x40_P2.54mm_Vertical
- removed P1: Host_Port, Connector_USB:USB_C_Receptacle_GCT_USB4085
- removed P2: Left_Peripheral, Connector_USB:USB_C_Receptacle_GCT_USB4085
- removed P3: Right_Peripheral, Connector_USB:USB_C_Receptacle_GCT_USB4085
- removed REF** (x4): MountingHole_2.2mm_M2_DIN965_Pad, MountingHole:MountingHole_2.2mm_M2_DIN965_Pad
- removed SW1: SW_Push, Button_Switch_SMD:SW_SPST_EVPBF
- removed U1: kb2040, footprints:kb2040
- removed U2: MCP23017_SO, Package_SO:SOIC-28W_7.5x17.9mm_P1.27mm
- removed U3: CH334R, Package_SO:QSOP-16_3.9x4.9mm_P0.635mm
- added J5: Conn_01x40_Socket, Connector_PinHeader_2.54mm:PinHeader_1x32_P2.54mm_Vertical, F.Cu at (67.5, 28.0)
- added J6: USB_Hub4_FDD, Connector_USB:USB_A_Molex_67643_Horizontal, F.Cu at (260.0, 13.0)
- added J7: USB_Hub3, Connector_USB:USB_A_Molex_67643_Horizontal, F.Cu at (240.0, 13.0)
- added J8: USB_Hub2, Connector_USB:USB_A_Molex_67643_Horizontal, F.Cu at (220.0, 13.0)
- added J9: Conn_01x16_Socket, Connector_PinHeader_2.54mm:PinHeader_1x32_P2.54mm_Vertical, F.Cu at (153.8, 28.0)
- added P4: Left_Peripheral, Connector_USB:USB_C_Receptacle_Amphenol_12401548E4-2A, F.Cu at (5.50, 15.0)
- added P5: Host_Port, Connector_USB:USB_C_Receptacle_Amphenol_12401548E4-2A, F.Cu at (280.0, 4.99)
- added P6: Right_Peripheral, Connector_USB:USB_C_Receptacle_Amphenol_12401548E4-2A, F.Cu at (294.5, 15.0)
- added SW2: SW_Push, Button_Switch_SMD:SW_SPST_EVPBF, F.Cu at (40.1, 7.00)
- added SW3: SW_Push, Button_Switch_SMD:SW_SPST_EVPBF, F.Cu at (52.9, 7.00)
- added SW4: SW_Push, Button_Switch_SMD:SW_SPST_EVPBF, F.Cu at (66.9, 7.00)
- added U4: PGA2350, pga2350:pga2350, F.Cu at (150.0, 12.7)
- added U5: CH334R, Package_SO:QSOP-16_3.9x4.9mm_P0.635mm, F.Cu at (259.4, 19.3)
Routing:
- net VBUS: track 419.0 -> 0.00 mm, vias 1 -> 0
- net MOSI: track 346.6 -> 0.00 mm, vias 3 -> 0
- net MISO: track 343.9 -> 0.00 mm
- net SDA: track 321.5 -> 0.00 mm, vias 1 -> 0
- net SCK: track 315.3 -> 0.00 mm, vias 1 -> 0
- net DM1+: track 145.1 -> 0.00 mm
- net DM1-: track 145.1 -> 0.00 mm
- net /Excelsior_PGA2350/SCK: track 0.00 -> 71.0 mm
- net /Excelsior_PGA2350/MOSI: track 0.00 -> 71.0 mm
- net RESET: track 69.1 -> 0.00 mm, vias 2 -> 0
- net /Excelsior_PGA2350/CS: track 0.00 -> 64.9 mm
- net /Excelsior_PGA2350/MISO: track 0.00 -> 64.8 mm
- net HOST_D-: track 59.6 -> 0.00 mm
- net HOST_D+: track 59.5 -> 0.00 mm
- net /Excelsior_PGA2350/GP06: track 0.00 -> 56.2 mm
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- added copper zone on B.Cu, net /Excelsior_PGA2350/GND
- added copper zone on F.Cu, net /Excelsior_PGA2350/GND
- removed copper zone on B.Cu, net GND
- removed copper zone on F.Cu, net GND
