File: pcb/excelsior.kicad_pcb (KiCad board)
At the start: 4 copper layers, 300 x 85 mm, 13 parts, among them J1 HDMI Breakout, J2 HDMI Breakout, J3 HDMI Breakout, J4 HDMI Breakout, J5 USB_A, J6 USB_A, J7 USB_A, SW1 SW_RST, SW2 SW_BOOT, SW3 SW_RST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

Commit message: Continue work on PCBs.
Parts:
- J1, J2, J3, J4: value HDMI Breakout -> Pogo Pin Connector; footprint excelsior:HDMI_Breakout -> Connector_PinHeader_2.54mm:PinHeader_1x12_P2.54mm_Vertical
- moved J3 65.7 mm to (3.50, 133.0)
- moved SW3 50.0 mm to (41.0, 104.5)
- moved U3 50.0 mm to (75.0, 117.5)
- moved J4 36.4 mm to (142.0, 103.9)
- moved J1 15.4 mm to (3.50, 31.7)
- moved J2 15.4 mm to (297.0, 3.53)
Connections:
- J1 pad 10: /Main Board/CS4 -> /Main Board/CS0
- J1 pad 11: /Main Board/INTA1 -> /Main Board/CS1
- J1 pad 12: /Main Board/CS5 -> /Main Board/CS2
- J2 pad 10: /Main Board/CS4 -> /Main Board/CS0
- J2 pad 11: /Main Board/INTA1 -> /Main Board/CS1
- J2 pad 12: /Main Board/CS5 -> /Main Board/CS2
- J3 pad 10: /Peripheral Board/CS4 -> /Peripheral Board/CS0
- J3 pad 11: /Peripheral Board/INTA1 -> /Peripheral Board/CS1
- J3 pad 12: /Peripheral Board/CS5 -> /Peripheral Board/CS2
- J4 pad 10: /Peripheral Board/CS4 -> /Peripheral Board/CS0
- J4 pad 11: /Peripheral Board/INTA1 -> /Peripheral Board/CS1
- J4 pad 12: /Peripheral Board/CS5 -> /Peripheral Board/CS2
Routing:
- net (no net): track 0.00 -> 1190.7 mm, vias 0 -> 8
- net /Peripheral Board/CS2: track 0.00 -> 290.2 mm, vias 0 -> 2
- net /Peripheral Board/CS0: track 0.00 -> 289.3 mm, vias 0 -> 2
- net /Peripheral Board/SCL: track 0.00 -> 183.4 mm, vias 0 -> 2
- net /Peripheral Board/SDA: track 0.00 -> 181.1 mm, vias 0 -> 2
- net /Peripheral Board/INTB1: track 0.00 -> 174.8 mm, vias 0 -> 2
- net /Peripheral Board/INTA1: track 0.00 -> 172.5 mm, vias 0 -> 2
- net /Peripheral Board/CS1: track 0.00 -> 144.3 mm, vias 0 -> 1
- net /Main Board/DP3: track 0.00 -> 102.9 mm
- net /Main Board/DN3: track 0.00 -> 102.8 mm
- net /Main Board/CS4: track 98.2 -> 0.00 mm
- net /Main Board/CS2: track 96.1 -> 0.00 mm
- net /Main Board/CS5: track 95.1 -> 0.00 mm
- net /Main Board/CS1: track 93.6 -> 0.00 mm
- net /Main Board/CS3: track 92.5 -> 0.00 mm
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Other:
- board size 300 x 85 mm -> 300 x 174.5 mm

Commit message: - Update main Readme. - Add folders for case CAD and KMK files. - In the PCBs, fix VBUS and GND being removed from connectors. - Add PCB readme.
Connections:
- J1 pad 1: /Main Board/MISO -> /Main Board/VBUS
- J1 pad 10: /Main Board/CS0 -> /Main Board/CS1
- J1 pad 11: /Main Board/CS1 -> /Main Board/CS2
- J1 pad 12: /Main Board/CS2 -> /Main Board/GND
- J1 pad 2: /Main Board/SCK -> /Main Board/MISO
- J1 pad 3: /Main Board/MOSI -> /Main Board/SCK
- J1 pad 4: /Main Board/SDA -> /Main Board/MOSI
- J1 pad 5: /Main Board/SCL -> /Main Board/SDA
- J1 pad 6: /Main Board/INTA1 -> /Main Board/SCL
- J1 pad 7: /Main Board/INTB1 -> /Main Board/INTA1
- J1 pad 8: /Main Board/INTA2 -> /Main Board/INTB1
- J1 pad 9: /Main Board/INTB2 -> /Main Board/CS0
- J2 pad 1: /Main Board/MISO -> /Main Board/VBUS
- J2 pad 10: /Main Board/CS0 -> /Main Board/CS1
- J2 pad 11: /Main Board/CS1 -> /Main Board/CS2
- J2 pad 12: /Main Board/CS2 -> /Main Board/GND
- J2 pad 2: /Main Board/SCK -> /Main Board/MISO
- J2 pad 3: /Main Board/MOSI -> /Main Board/SCK
- J2 pad 4: /Main Board/SDA -> /Main Board/MOSI
- J2 pad 5: /Main Board/SCL -> /Main Board/SDA
- J2 pad 6: /Main Board/INTA1 -> /Main Board/SCL
- J2 pad 7: /Main Board/INTB1 -> /Main Board/INTA1
- J2 pad 8: /Main Board/INTA2 -> /Main Board/INTB1
- J2 pad 9: /Main Board/INTB2 -> /Main Board/CS0
- J3 pad 1: /Peripheral Board/MISO -> /Peripheral Board/VBUS
- J3 pad 10: /Peripheral Board/CS0 -> /Peripheral Board/CS1
- J3 pad 11: /Peripheral Board/CS1 -> /Peripheral Board/CS2
- J3 pad 12: /Peripheral Board/CS2 -> /Peripheral Board/GND
- J3 pad 2: /Peripheral Board/SCK -> /Peripheral Board/MISO
- J3 pad 3: /Peripheral Board/MOSI -> /Peripheral Board/SCK
- J3 pad 4: /Peripheral Board/SDA -> /Peripheral Board/MOSI
- J3 pad 5: /Peripheral Board/SCL -> /Peripheral Board/SDA
- J3 pad 6: /Peripheral Board/INTA1 -> /Peripheral Board/SCL
- J3 pad 7: /Peripheral Board/INTB1 -> /Peripheral Board/INTA1
- J3 pad 8: /Peripheral Board/INTA2 -> /Peripheral Board/INTB1
- J3 pad 9: /Peripheral Board/INTB2 -> /Peripheral Board/CS0
- J4 pad 1: /Peripheral Board/MISO -> /Peripheral Board/VBUS
- J4 pad 10: /Peripheral Board/CS0 -> /Peripheral Board/CS1
- J4 pad 11: /Peripheral Board/CS1 -> /Peripheral Board/CS2
- J4 pad 12: /Peripheral Board/CS2 -> /Peripheral Board/GND
- J4 pad 2: /Peripheral Board/SCK -> /Peripheral Board/MISO
- J4 pad 3: /Peripheral Board/MOSI -> /Peripheral Board/SCK
- J4 pad 4: /Peripheral Board/SDA -> /Peripheral Board/MOSI
- J4 pad 5: /Peripheral Board/SCL -> /Peripheral Board/SDA
- J4 pad 6: /Peripheral Board/INTA1 -> /Peripheral Board/SCL
- J4 pad 7: /Peripheral Board/INTB1 -> /Peripheral Board/INTA1
- J4 pad 8: /Peripheral Board/INTA2 -> /Peripheral Board/INTB1
- J4 pad 9: /Peripheral Board/INTB2 -> /Peripheral Board/CS0
Routing:
- net (no net): track 1190.7 -> 0.00 mm, vias 8 -> 0
- net /Main Board/CS2: track 0.00 -> 363.7 mm, vias 0 -> 2
- net /Main Board/CS0: track 0.00 -> 361.0 mm, vias 0 -> 2
- net /Main Board/CS1: track 0.00 -> 359.2 mm, vias 0 -> 2
- net /Main Board/INTB1: track 0.00 -> 353.7 mm, vias 0 -> 2
- net /Main Board/INTA1: track 0.00 -> 351.6 mm, vias 0 -> 2
- net /Main Board/SCL: track 0.00 -> 350.0 mm, vias 0 -> 2
- net /Main Board/MISO: track 0.00 -> 349.1 mm, vias 0 -> 2
- net /Main Board/SDA: track 0.00 -> 348.4 mm, vias 0 -> 2
- net /Main Board/MOSI: track 0.00 -> 347.4 mm, vias 0 -> 2
- net /Main Board/SCK: track 0.00 -> 346.4 mm, vias 0 -> 2
- net /Peripheral Board/MOSI: track 0.00 -> 151.1 mm, vias 0 -> 1
- net /Peripheral Board/SCK: track 0.00 -> 149.9 mm, vias 0 -> 1
- net /Peripheral Board/MISO: track 0.00 -> 148.5 mm, vias 0 -> 1
- net /Peripheral Board/CS0: track 289.3 -> 162.1 mm, vias 2 -> 1
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
Commit message: - Change pogo pin connectors on opposite sides from rotated to mirrored. - Add lots of firmware code. - Add VSCode settings to gitignore.
Parts:
- moved J3 29.1 mm to (3.50, 103.9), turned to 0 degrees
- moved J1 28.2 mm to (3.50, 3.53), turned to 0 degrees
Routing:
- net /Main Board/VBUS: track 365.2 -> 392.0 mm
- net /Main Board/CS2: track 363.7 -> 339.8 mm, vias 2 -> 1
- net /Main Board/CS1: track 359.2 -> 339.0 mm, vias 2 -> 1
- net /Main Board/CS0: track 361.0 -> 344.3 mm, vias 2 -> 1
- net /Peripheral Board/MISO: track 148.5 -> 163.4 mm, vias 1 -> 0
- net /Peripheral Board/CS2: track 166.8 -> 151.9 mm, vias 1 -> 0
- net /Main Board/INTB1: track 353.7 -> 340.7 mm, vias 2 -> 1
- net /Peripheral Board/SDA: track 176.1 -> 188.7 mm, vias 2 -> 1
- net /Peripheral Board/SCK: track 149.9 -> 162.1 mm, vias 1 -> 0
- net /Peripheral Board/CS1: track 164.4 -> 153.2 mm, vias 1 -> 0
- net /Peripheral Board/MOSI: track 151.1 -> 160.9 mm, vias 1 -> 0
- net /Main Board/INTA1: track 351.6 -> 342.2 mm, vias 2 -> 1
- net /Peripheral Board/SCL: track 179.3 -> 188.4 mm, vias 2 -> 1
- net /Peripheral Board/CS0: track 162.1 -> 154.5 mm, vias 1 -> 0
- net /Main Board/SCL: track 350.0 -> 344.1 mm, vias 2 -> 1
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