File: pcb/excelsior.kicad_sch (KiCad schematic)
At the start: 0 parts

Commit message: Continue work on PCBs.
Other:
- added sheet Main Board (main_board.kicad_sch)
- added sheet Peripheral Board (peripheral_board.kicad_sch)
Changed lines of the file:
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@@
 	(generator_version "9.0")
 	(paper "A4")
+	(sheet
+		(at 43.18 46.99)
+		(size 12.7 3.81)
+		(exclude_from_sim no)
+		(in_bom yes)
+		(on_board yes)
+		(dnp no)
+		(fields_autoplaced yes)
+		(stroke
+			(width 0.1524)
+			(type solid)
+		)
+		(fill
+			(color 0 0 0 0.0000)
+		)
+		(property "Sheetname" "Main Board"
+			(at 43.18 46.2784 0)
+			(effects
+				(font
+					(size 1.27 1.27)
+				)
+				(justify left bottom)
+			)
+		)
+		(property "Sheetfile" "main_board.kicad_sch"
+			(at 43.18 51.3846 0)
+			(effects
+				(font
+					(size 1.27 1.27)
+				)
+				(justify left top)
+			)
+		)
+		(instances
+			(project "excelsior"
+				(path "/70e7ac93-e728-47cd-97d6-fe8c6ae34c94"
+					(page "2")
+				)
+			)
+		)
+	)
+	(sheet
+		(at 85.09 45.72)
+		(size 12.7 3.81)
+		(exclude_from_sim no)
+		(in_bom yes)
+		(on_board yes)
+		(dnp no)
+		(fields_autoplaced yes)
+		(stroke
+			(width 0.1524)
+			(type solid)
+		)
+		(fill
+			(color 0 0 0 0.0000)
+		)
+		(property "Sheetname" "Peripheral Board"
+			(at 85.09 45.0084 0)
+			(effects
+				(font
+					(size 1.27 1.27)
+				)
+				(justify left bottom)
+			)
+		)
+		(property "Sheetfile" "peripheral_board.kicad_sch"
+			(at 85.09 50.1146 0)
+			(effects
+				(font
+					(size 1.27 1.27)
+				)
+				(justify left top)
+			)
+		)
+		(instances
+			(project "excelsior"
+				(path "/70e7ac93-e728-47cd-97d6-fe8c6ae34c94"
+					(page "3")
+				)
+			)
+		)
+	)
 	(sheet_instances
 		(path "/"
