File: pcb/excelsior_pga2350.kicad_sch (KiCad schematic)
At the start: 13 parts, among them J5 Conn_01x40_Socket, J6 USB_Hub4_FDD, J7 USB_Hub3, J8 USB_Hub2, J9 Conn_01x16_Socket, P4 Left_Peripheral, P5 Host_Port, P6 Right_Peripheral, SW2 SW_Push, SW3 SW_Push, SW4 SW_Push, U4 PGA2350, U5 CH334R

Commit message: Continue work on PCBs.
Parts:
- J5: footprint Connector_PinHeader_2.54mm:PinHeader_1x40_P2.54mm_Vertical -> Connector_PinHeader_2.54mm:PinHeader_1x32_P2.54mm_Vertical; symbol Connector:Conn_01x40_Socket -> Connector:Conn_01x32_Socket
- J9: footprint (none) -> Connector_PinHeader_2.54mm:PinHeader_1x32_P2.54mm_Vertical; symbol Connector:Conn_01x16_Socket -> Connector:Conn_01x32_Socket
- P4, P5, P6: footprint Connector_USB:USB_C_Receptacle_GCT_USB4085 -> Connector_USB:USB_C_Receptacle_Amphenol_12401548E4-2A
- U4: footprint (none) -> pga2350:pga2350
Connections:
- net IO_00 is gone; now on net INTA: J5.3 (Pin_3), U4.00 (GP00)
- net IO_01 is gone; now on net INTB: J5.4 (Pin_4), U4.01 (GP01)
- net GND: now also J5.1 (Pin_1), J5.17 (Pin_17), J5.25 (Pin_25), J5.9 (Pin_9), J9.1 (Pin_1), J9.17 (Pin_17), J9.25 (Pin_25), J9.26 (Pin_26), J9.27 (Pin_27), J9.28 (Pin_28), J9.29 (Pin_29), J9.30 (Pin_30), J9.32 (Pin_32), J9.9 (Pin_9); no longer J5.10 (Pin_10), J5.18 (Pin_18), J5.2 (Pin_2), J5.31 (Pin_31), J5.39 (Pin_39)
- net MISO: now also P4.A6 (D+), P4.B6 (D+), P6.A6 (D+), P6.B6 (D+); no longer P4.A7 (D-), P4.B7 (D-), P6.A7 (D-), P6.B7 (D-)
- net MOSI: now also P4.A7 (D-), P4.B7 (D-), P6.A7 (D-), P6.B7 (D-); no longer P4.A6 (D+), P4.B6 (D+), P6.A6 (D+), P6.B6 (D+)
- net VBUS: now also J5.2 (Pin_2), U4.3EN (3V3_EN); no longer J5.1 (Pin_1), J5.40 (Pin_40)
- net GP40: now reaches J9.16 (Pin_16)
- net GP40: now also U4.40 (GP40)
- net IO_06 renamed GP06
- net GP06: now also J5.10 (Pin_10); no longer J5.9 (Pin_9)
- net IO_07 renamed GP07
- net IO_08 renamed GP08
- net IO_09 renamed GP09
- net IO_10 renamed GP10
- net IO_11 renamed GP11
- net IO_12 renamed GP12
- net IO_13 renamed GP13
- net GP13: now also J5.18 (Pin_18); no longer J5.17 (Pin_17)
- net IO_14 renamed GP14
- net IO_15 renamed GP15
- net IO_16 renamed GP16
- net IO_17 renamed GP17
- net IO_18 renamed GP18
- net IO_19 renamed GP19
- net IO_20 renamed GP20
- net GP20: now also J5.26 (Pin_26); no longer J5.25 (Pin_25)
- net IO_21 renamed GP21
- net GP21: now also J5.27 (Pin_27); no longer J5.26 (Pin_26)
- net IO_22 renamed GP22
- net GP22: now also J5.28 (Pin_28); no longer J5.27 (Pin_27)
- net IO_23 renamed GP23
- net GP23: now also J5.29 (Pin_29); no longer J5.28 (Pin_28)
- net IO_24 renamed GP24
- net GP24: now also J5.30 (Pin_30); no longer J5.29 (Pin_29)
- net IO_25 renamed GP25
- net GP25: now also J5.31 (Pin_31); no longer J5.30 (Pin_30)
- net IO_26 renamed GP26
- net IO_27 renamed GP27
- net GP27: now also J9.2 (Pin_2); no longer J5.33 (Pin_33)
- net IO_28 renamed GP28
- net GP28: now also J9.3 (Pin_3); no longer J5.34 (Pin_34)
- net IO_29 renamed GP29
- net GP29: now also J9.4 (Pin_4); no longer J5.35 (Pin_35)
- net IO_30 renamed GP30
- net GP30: now also J9.5 (Pin_5); no longer J5.36 (Pin_36)
- net IO_31 renamed GP31
- net GP31: now also J9.6 (Pin_6); no longer J5.37 (Pin_37)
- net IO_32 renamed GP32
- net GP32: now also J9.7 (Pin_7); no longer J5.38 (Pin_38)
- net IO_33 renamed GP33
- net GP33: now also J9.8 (Pin_8); no longer J9.15 (Pin_15)
- net IO_34 renamed GP34
- net GP34: now also J9.10 (Pin_10); no longer J9.14 (Pin_14)
- net IO_35 renamed GP35
- net GP35: now also J9.11 (Pin_11); no longer J9.13 (Pin_13)
- net IO_36 renamed GP36
- net IO_37 renamed GP37
- net GP37: now also J9.13 (Pin_13); no longer J9.11 (Pin_11)
- net IO_38 renamed GP38
- net GP38: now also J9.14 (Pin_14); no longer J9.10 (Pin_10)
- net IO_39 renamed GP39
- net GP39: now also J9.15 (Pin_15); no longer J9.9 (Pin_9)
- removed net IO_40: J9.8 (Pin_8), U4.40 (GP40)
- net IO_41 renamed GP41
- net GP41: now also J9.18 (Pin_18); no longer J9.7 (Pin_7)
- net IO_42 renamed GP42
- net GP42: now also J9.19 (Pin_19); no longer J9.6 (Pin_6)
- net IO_43 renamed GP43
- net GP43: now also J9.20 (Pin_20); no longer J9.5 (Pin_5)
- net IO_44 renamed GP44
- net GP44: now also J9.21 (Pin_21); no longer J9.4 (Pin_4)
- net IO_45 renamed GP45
- net GP45: now also J9.22 (Pin_22); no longer J9.3 (Pin_3)
- net IO_46 renamed GP46
- net GP46: now also J9.23 (Pin_23); no longer J9.2 (Pin_2)
- net IO_47 renamed GP47
- net GP47: now also J9.24 (Pin_24); no longer J9.1 (Pin_1)
- new net 3V3: J9.31 (Pin_31), U4.3V3
- no-connect marks 29 -> 26
