File: pcb/v0.0.1/excelsior_pga2350.kicad_sch (KiCad schematic)
At the start: 13 parts, among them J5 Conn_01x40_Socket, J6 USB_Hub4_FDD, J7 USB_Hub3, J8 USB_Hub2, J9 Conn_01x16_Socket, P4 Left_Peripheral, P5 Host_Port, P6 Right_Peripheral, SW2 SW_Push, SW3 SW_Push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

Commit message: Fresh start on PCBs.
Connections:
- net CS: now also P4.B3 (TX2-), P6.B3 (TX2-); no longer P4.A2 (TX1+), P6.A2 (TX1+)
- net INTA: now also P4.B10 (RX1-), P6.B10 (RX1-); no longer P4.A11 (RX2+), P6.A11 (RX2+)
- net INTB: now also P4.A11 (RX2+), P4.B11 (RX1+), P6.A11 (RX2+), P6.B11 (RX1+); no longer P4.B2 (TX2+), P4.B3 (TX2-), P6.B2 (TX2+), P6.B3 (TX2-)
- net SCK: now also P4.A2 (TX1+), P4.B2 (TX2+), P6.A2 (TX1+), P6.B2 (TX2+); no longer P4.B10 (RX1-), P4.B11 (RX1+), P6.B10 (RX1-), P6.B11 (RX1+)
