File: pcb/current_version/mcp23s17_breakout/mcp23s17_breakout.kicad_sch (KiCad schematic)
At the start: 0 parts

Commit message: Add breakout boards for MCP23S17 and HDMI connector.
Parts:
- added J1, J2: Conn_01x14, Connector_PinHeader_2.54mm:PinHeader_1x14_P2.54mm_Vertical, symbol Connector_Generic:Conn_01x14
- added U1: MCP23017_SO, Package_SO:SOIC-28W_7.5x17.9mm_P1.27mm, symbol Interface_Expansion:MCP23S17_SO
Connections:
- new net A0: J2.6 (Pin_6), U1.15 (A0)
- new net A1: J2.5 (Pin_5), U1.16 (A1)
- new net A2: J2.4 (Pin_4), U1.17 (A2)
- new net CS: J1.5 (Pin_5), U1.11 (~{CS})
- new net GND: J1.1 (Pin_1), U1.10 (VSS)
- new net GPA0: J1.7 (Pin_7), U1.21 (GPA0)
- new net GPA1: J1.8 (Pin_8), U1.22 (GPA1)
- new net GPA2: J1.9 (Pin_9), U1.23 (GPA2)
- new net GPA3: J1.10 (Pin_10), U1.24 (GPA3)
- new net GPA4: J1.11 (Pin_11), U1.25 (GPA4)
- new net GPA5: J1.12 (Pin_12), U1.26 (GPA5)
- new net GPA6: J1.13 (Pin_13), U1.27 (GPA6)
- new net GPA7: J1.14 (Pin_14), U1.28 (GPA7)
- new net GPB0: J2.7 (Pin_7), U1.1 (GPB0)
- new net GPB1: J2.8 (Pin_8), U1.2 (GPB1)
- new net GPB2: J2.9 (Pin_9), U1.3 (GPB2)
- new net GPB3: J2.10 (Pin_10), U1.4 (GPB3)
- new net GPB4: J2.11 (Pin_11), U1.5 (GPB4)
- new net GPB5: J2.12 (Pin_12), U1.6 (GPB5)
- new net GPB6: J2.13 (Pin_13), U1.7 (GPB6)
- new net GPB7: J2.14 (Pin_14), U1.8 (GPB7)
- new net INTA: J2.2 (Pin_2), U1.20 (INTA)
- new net INTB: J2.3 (Pin_3), U1.19 (INTB)
- new net RST: J1.6 (Pin_6), U1.18 (~{RESET})
- new net SCK: J1.4 (Pin_4), U1.12 (SCK)
- new net SI: J1.3 (Pin_3), U1.13 (SI)
- new net SO: J1.2 (Pin_2), U1.14 (SO)
- new net VBUS: J2.1 (Pin_1), U1.9 (VDD)
