File: pcb/mcp23s17_breakout/mcp23s17_breakout.kicad_pcb (KiCad board)
At the start: 2 copper layers, 26 x 36 mm, 3 parts, among them J1 Conn_01x14, J2 Conn_01x14, U1 MCP23017_SO

Commit message: Continue work on PCBs.
Parts:
- moved J2 40.2 mm to (23.0, 33.0), turned to 180 degrees
- moved J1 40.1 mm to (0.14, -0.02), turned to 0 degrees
- moved U1 1.36 mm to (11.6, 17.2), turned to 180 degrees
Connections:
- J1 pad 10: /GPA3 -> /GPA4
- J1 pad 11: /GPA4 -> /GPA5
- J1 pad 12: /GPA5 -> /GPA6
- J1 pad 13: /GPA6 -> /GPA7
- J2 pad 14: /GPB7 -> /VBUS
